Commit message: Corrected 3d design

File: auto_tractor/urdf/auto_tractor.urdf (robot description, URDF)
Before this commit: robot auto_tractor, 5 links, 4 joints
Links:
- removed link Front_Left
- removed link Front_Right
- removed link Rear_Left
- removed link Rear_Right
- added link Front_left, mass 100; collision mesh filename=package://auto_tractor/meshes/Front_left.STL; visual mesh filename=package://auto_tractor/meshes/Front_left.STL
- added link Front_right, mass 100; collision mesh filename=package://auto_tractor/meshes/Front_right.STL; visual mesh filename=package://auto_tractor/meshes/Front_right.STL
- added link Rear_left, mass 100; collision mesh filename=package://auto_tractor/meshes/Rear_left.STL; visual mesh filename=package://auto_tractor/meshes/Rear_left.STL
- added link Rear_right, mass 100; collision mesh filename=package://auto_tractor/meshes/Rear_right.STL; visual mesh filename=package://auto_tractor/meshes/Rear_right.STL
- link base_link: mass 2950 -> 2890
Joints:
- joint FL: child Front_Left -> Front_left; origin xyz=0.91935 -0.78962 -0.29152 rpy=0.33919 0.0051747 -0.016201 -> xyz=0.92099 -0.63407 -0.53606 rpy=0.34375 0 0
- joint FR: child Front_Right -> Front_right; origin xyz=0.92252 0.76364 -0.29088 rpy=0.33919 0.0051747 -0.016201 -> xyz=0.92109 0.83018 -0.011833 rpy=0.34375 0 0
- joint RL: child Rear_Left -> Rear_left; origin xyz=-1.3467 -0.78264 -0.10971 rpy=0.33919 0.0051747 -0.016201 -> xyz=-1.3428 -0.81744 -0.40911 rpy=0.34375 0 0
- joint RR: child Rear_Right -> Rear_right; origin xyz=-1.341 0.80939 -0.10956 rpy=0.33919 0.0051747 -0.016201 -> xyz=-1.3428 0.8161 0.17548 rpy=0.34375 -0.00020469 -7.3256E-05

Commit message: Update auto_tractor.urdf

File: auto_tractor/urdf/auto_tractor.urdf (robot description, URDF)
Before this commit: robot auto_tractor, 5 links, 4 joints
Links:
- link Front_left: mass 100 -> 0.208066209258392
- link Front_right: mass 100 -> 0.208066209260515
- link Rear_left: mass 100 -> 0.245765324492604
- link Rear_right: mass 100 -> 0.245765324492615
- link base_link: mass 2890 -> 58.1363480593461
Joints:
- joint FL: axis 0 1 0 -> 0.0066741 0.99964 -0.026176; origin xyz=0.92099 -0.63407 -0.53606 rpy=0.34375 0 0 -> xyz=0.92175 -0.77667 -0.2912 rpy=0 0.00021738 0
- joint FR: axis 0 1 0 -> 0.99963 -0.0077313 -0.026176; origin xyz=0.92109 0.83018 -0.011833 rpy=0.34375 0 0 -> xyz=0.92021 0.7786 -0.29113 rpy=0.040824 -0.00030073 1.5708
- joint RL: axis 0 1 0 -> -0.0010575 1 0; origin xyz=-1.3428 -0.81744 -0.40911 rpy=0.34375 0 0 -> xyz=-1.3419 -0.90892 -0.10944 rpy=0 0.00021738 0
- joint RR: axis 0 1 0 -> -0.0010572 1 0; origin xyz=-1.3428 0.8161 0.17548 rpy=0.34375 -0.00020469 -7.3256E-05 -> xyz=-1.3437 0.82608 -0.10955 rpy=0 0 0

Commit message: Update auto_tractor.urdf

File: auto_tractor/urdf/auto_tractor.urdf (robot description, URDF)
Before this commit: robot auto_tractor, 5 links, 4 joints
Links:
- link Front_left: mass 0.208066209258392 -> 2890
- link Front_right: mass 0.208066209260515 -> 2890
- link Rear_left: mass 0.245765324492604 -> 2890
- link Rear_right: mass 0.245765324492615 -> 2890
- link base_link: mass 58.1363480593461 -> 2890
Joints:
- joint FL: axis 0.0066741 0.99964 -0.026176 -> -0.0077993 0.99963 -0.026196; origin xyz=0.92175 -0.77667 -0.2912 rpy=0 0.00021738 0 -> xyz=0.92106 -0.77764 -0.29107 rpy=0.05236 0 0
- joint FR: axis 0.99963 -0.0077313 -0.026176 -> -0.0077313 -0.99963 -0.026176; origin xyz=0.92021 0.7786 -0.29113 rpy=0.040824 -0.00030073 1.5708 -> xyz=0.92111 0.77762 -0.29104 rpy=-0.05236 0 0
- joint RL: axis -0.0010575 1 0 -> 0 1 0; origin xyz=-1.3419 -0.90892 -0.10944 rpy=0 0.00021738 0 -> xyz=-1.3427 -0.8025 -0.10985 rpy=0 0 0
- joint RR: axis -0.0010572 1 0 -> 0 1 0; origin xyz=-1.3437 0.82608 -0.10955 rpy=0 0 0 -> xyz=-1.3427 0.8025 -0.10985 rpy=0 0 0

Commit message: sensors added

File: auto_tractor/urdf/auto_tractor.urdf (robot description, URDF)
Before this commit: robot auto_tractor, 5 links, 4 joints
Links:
- added link ultrasonic_link, mass 0.01; collision cylinder length=0.02 radius=0.01; visual cylinder length=0.02 radius=0.01
Joints:
- added joint ultrasonic_joint: type fixed, parent base_link, child ultrasonic_link, origin xyz=1.8 0 0.1 rpy=0 0 0

Commit message: sensors position updated

File: auto_tractor/urdf/auto_tractor.urdf (robot description, URDF)
Before this commit: robot auto_tractor, 6 links, 5 joints
Joints:
- joint ultrasonic_joint: origin xyz=1.8 0 0.1 rpy=0 0 0 -> xyz=0 0 0 rpy=0 0 0

Commit message: velocity controller topics added for each wheel joint

File: auto_tractor/urdf/auto_tractor.urdf (robot description, URDF)
Before this commit: robot auto_tractor, 6 links, 5 joints
Joints:
- joint FL: limit (none) -> lower=0 upper=0 effort=100000 velocity=1
- joint FR: limit (none) -> lower=0 upper=0 effort=100000 velocity=1
- joint RL: limit (none) -> lower=0 upper=0 effort=100000 velocity=1
- joint RR: limit (none) -> lower=0 upper=0 effort=100000 velocity=1

Commit message: velocity contorllers updated

File: auto_tractor/urdf/auto_tractor.urdf (robot description, URDF)
Before this commit: robot auto_tractor, 6 links, 5 joints
Joints:
- joint FL: limit lower=0 upper=0 effort=100000 velocity=1 -> (none)
- joint FR: limit lower=0 upper=0 effort=100000 velocity=1 -> (none)
- joint RL: limit lower=0 upper=0 effort=100000 velocity=1 -> (none)
- joint RR: limit lower=0 upper=0 effort=100000 velocity=1 -> (none)

Commit message: velocity topics added for each wheel

File: auto_tractor/urdf/auto_tractor.urdf (robot description, URDF)
Before this commit: robot auto_tractor, 6 links, 5 joints
Joints:
- joint FL: axis -0.0077993 0.99963 -0.026196 -> 0 1 0; origin xyz=0.92106 -0.77764 -0.29107 rpy=0.05236 0 0 -> xyz=0.92106 -0.77764 -0.29107 rpy=-0.05236 0 0
- joint FR: axis -0.0077313 -0.99963 -0.026176 -> 0 1 0; origin xyz=0.92111 0.77762 -0.29104 rpy=-0.05236 0 0 -> xyz=0.92106 0.77764 -0.29104 rpy=0.05236 0 0

Commit message: Controller and publishers added for all joints

File: auto_tractor/urdf/auto_tractor.urdf (robot description, URDF)
Before this commit: robot auto_tractor, 6 links, 5 joints
Links:
- added link front_left_steering_link, mass 50.0; collision cylinder length=0.05 radius=0.1; visual cylinder length=0.05 radius=0.1
- added link front_right_steering_link, mass 50.0; collision cylinder length=0.05 radius=0.1; visual cylinder length=0.05 radius=0.1
- link Front_left: mass 2890 -> 578
- link Front_right: mass 2890 -> 578
- link Rear_left: mass 2890 -> 578
- link Rear_right: mass 2890 -> 578
- link base_link: mass 2890 -> 578
Joints:
- added joint front_left_steering_joint: type revolute, parent base_link, child front_left_steering_link, origin xyz=0.92106 -0.77764 -0.29107 rpy=0 0 0, axis 0 0 1, limit lower=-0.6 upper=0.6 effort=10000 velocity=1000
- added joint front_right_steering_joint: type revolute, parent base_link, child front_right_steering_link, origin xyz=0.92106 0.77764 -0.29107 rpy=0 0 0, axis 0 0 1, limit lower=-0.6 upper=0.6 effort=10000 velocity=1000
- joint FL: origin xyz=0.92106 -0.77764 -0.29107 rpy=-0.05236 0 0 -> xyz=0 0 0 rpy=-0.05236 0 0; parent base_link -> front_left_steering_link
- joint FR: origin xyz=0.92106 0.77764 -0.29104 rpy=0.05236 0 0 -> xyz=0 0 0 rpy=0.05236 0 0; parent base_link -> front_right_steering_link
